File: pcbs/lowkey36c.kicad_pcb (KiCad board)
At the start: 2 copper layers, 265.3 x 81 mm, 76 parts

Commit message: add component submodules and update pcb files
Parts:
- added LMH1: MountingHole_2.2mm_M2_DIN965_Pad_TopBottom, MountingHole:MountingHole_2.2mm_M2_DIN965_Pad_TopBottom, F.Cu at (30.1, 65.0)
- added LMH2: MountingHole_2.2mm_M2_DIN965_Pad_TopBottom, MountingHole:MountingHole_2.2mm_M2_DIN965_Pad_TopBottom, F.Cu at (27.1, 124.1)
- added LMH3: MountingHole_2.2mm_M2_DIN965_Pad_TopBottom, MountingHole:MountingHole_2.2mm_M2_DIN965_Pad_TopBottom, F.Cu at (110.3, 109.3)
- added LS1: SSSS811101, mg_pwr_sw:SW_SSSS811101, F.Cu at (39.6, 125.7)
- added REF**: mousebites 1mm, PCM_marbastlib-various:mousebites_1mm, F.Cu at (156.3, 132.4)
- added REF**: mousebites 1mm, PCM_marbastlib-various:mousebites_1mm, F.Cu at (106.9, 76.5)
- added REF**: mousebites 1mm, PCM_marbastlib-various:mousebites_1mm, F.Cu at (142.7, 132.5)
- added REF**: mousebites 1mm, PCM_marbastlib-various:mousebites_1mm, F.Cu at (192.1, 76.5)
- added RMH1: MountingHole_2.2mm_M2_DIN965_Pad_TopBottom, MountingHole:MountingHole_2.2mm_M2_DIN965_Pad_TopBottom, F.Cu at (269.7, 65.0)
- added RMH2: MountingHole_2.2mm_M2_DIN965_Pad_TopBottom, MountingHole:MountingHole_2.2mm_M2_DIN965_Pad_TopBottom, F.Cu at (271.0, 124.1)
- added RMH3: MountingHole_2.2mm_M2_DIN965_Pad_TopBottom, MountingHole:MountingHole_2.2mm_M2_DIN965_Pad_TopBottom, F.Cu at (188.7, 109.3)
- added RS1: SSSS811101, mg_pwr_sw:SW_SSSS811101, F.Cu at (259.9, 125.7)
- LJ1, RJ1: moved to B.Cu
- LU1, RU1: value Seeeduino Xiao nRF52840 -> XIAO-nRF52840-SMD; footprint PCM_marbastlib-xp-promicroish:Xiao_nRF52840_ACH -> kleeb_mcu:xiao-ble-smd-cutout; moved to F.Cu
- moved RJ1 51.9 mm to (211.8, 119.0), turned to 0 degrees
- moved LJ1 45.0 mm to (83.6, 119.4), turned to 0 degrees
- moved LD18 14.5 mm to (140.3, 128.2), turned to 70 degrees
- moved RD18 14.5 mm to (158.7, 128.1), turned to -70 degrees
- moved LSW18 12.9 mm to (135.8, 126.5), turned to -110 degrees
- moved RSW18 12.9 mm to (163.3, 126.4), turned to 110 degrees
- moved LD17 9.31 mm to (124.4, 122.1), turned to 70 degrees
- moved RD17 9.21 mm to (174.9, 122.2), turned to -70 degrees
- moved RSW17 7.94 mm to (179.3, 120.6), turned to 110 degrees
- moved LSW17 7.94 mm to (119.7, 120.6), turned to -110 degrees
- moved LU1 6.48 mm to (61.9, 116.8), turned to 180 degrees
- moved RU1 6.48 mm to (237.1, 116.8), turned to 180 degrees
Connections:
- LU1 pad 13: unconnected-(LU1-P1.13-Pad13) -> LGND
- LU1 pad 15: LGND -> +LBAT
- LU1 pad 16: +LBAT -> LGND
- LU1 pad 9: LGND -> unconnected-(LU1-P1.13_D8_SCK-Pad9)
- RU1 pad 13: unconnected-(RU1-P1.13-Pad13) -> RGND
- RU1 pad 15: RGND -> +RBAT
- RU1 pad 16: +RBAT -> RGND
- RU1 pad 9: RGND -> unconnected-(RU1-P1.13_D8_SCK-Pad9)
Other:
- board size 265.3 x 81 mm -> 265.3 x 94.8 mm
